File: Rev. 0/Eagle/C64_KernalSw_16k.brd (EAGLE design)
At the start: 22 x 45 mm, 13 parts, among them IC1 M27C512-DIP28, IC2 23128SOCKET, IC3 74HCT08D

Commit message: Silk Screen Update
Parts:
- added U$21: OPEN_SOURCE_HW, Logo:OPENHW
- added U$22: (no value), Logo:SVEN_TAG
Other:
- board text added: "100n"
- board text added: "10k"
- board text added: "LS08"
- board text added: "http://github.com/ svenpetersen1965"
Changed lines of the file:
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@@
 <?xml version="1.0" encoding="utf-8"?>
 <!DOCTYPE eagle SYSTEM "eagle.dtd">
-<eagle version="9.2.2">
+<eagle version="9.5.2">
 <drawing>
 <settings>
@@
 <layer number="21" name="tPlace" color="7" fill="1" visible="yes" active="yes"/>
 <layer number="22" name="bPlace" color="7" fill="1" visible="no" active="yes"/>
-<layer number="23" name="tOrigins" color="15" fill="1" visible="no" active="yes"/>
+<layer number="23" name="tOrigins" color="15" fill="1" visible="yes" active="yes"/>
 <layer number="24" name="bOrigins" color="15" fill="1" visible="no" active="yes"/>
 <layer number="25" name="tNames" color="7" fill="1" visible="yes" active="yes"/>
@@
 <layer number="45" name="Holes" color="7" fill="1" visible="no" active="yes"/>
 <layer number="46" name="Milling" color="3" fill="1" visible="no" active="yes"/>
-<layer number="47" name="Measures" color="7" fill="1" visible="no" active="yes"/>
+<layer number="47" name="Measures" color="7" fill="1" visible="yes" active="yes"/>
 <layer number="48" name="Document" color="5" fill="1" visible="yes" active="yes"/>
 <layer number="49" name="Reference" color="7" fill="1" visible="no" active="yes"/>
@@
 <layer number="250" name="Descript" color="7" fill="1" visible="no" active="no"/>
 <layer number="251" name="SMDround" color="7" fill="1" visible="no" active="no"/>
+<layer number="252" name="BR-BS" color="7" fill="1" visible="no" active="yes"/>
+<layer number="253" name="BR-LS" color="7" fill="1" visible="no" active="yes"/>
 <layer number="254" name="OrgLBR" color="7" fill="1" visible="no" active="no"/>
 <layer number="255" name="Accent" color="7" fill="1" visible="no" active="yes"/>
@@
 C64 short board</text>
 <text x="11.27125" y="3.81" size="1.1684" layer="21" ratio="12" rot="R90">Rev. 0</text>
-<text x="8.41375" y="6.19125" size="1.6764" layer="22" ratio="12" rot="MR90">Kernal Adapt/Sw  Rev. 0
+<text x="10.31875" y="1.27" size="1.27" layer="22" ratio="12" rot="MR90">Kernal Adapt/Sw  Rev. 0
 C64 short board</text>
+<text x="13.0175" y="23.1775" size="1.016" layer="21" ratio="12" rot="R90">LS08</text>
+<text x="7.3025" y="27.94" size="1.016" layer="21" ratio="12" rot="R90">10k</text>
+<text x="8.41375" y="17.145" size="1.016" layer="21" ratio="12" rot="R90">10k</text>
+<text x="10.795" y="17.30375" size="1.016" layer="21" ratio="12" rot="R90">10k</text>
+<text x="11.7475" y="33.3375" size="1.016" layer="21" ratio="12">100n</text>
+<text x="6.0325" y="1.42875" size="1.016" layer="22" ratio="12" rot="MR90">http://github.com/
+svenpetersen1965</text>
+<text x="13.6525" y="35.40125" size="1.27" layer="22" ratio="12" rot="MR0">GND</text>
+<wire x1="9.2075" y1="36.67125" x2="9.2075" y2="36.03625" width="0.127" layer="22"/>
+<wire x1="9.2075" y1="36.03625" x2="10.16" y2="36.03625" width="0.127" layer="22"/>
+<wire x1="13.97" y1="36.03625" x2="14.605" y2="36.03625" width="0.127" layer="22"/>
+<wire x1="14.605" y1="36.03625" x2="14.605" y2="36.67125" width="0.127" layer="22"/>
+<wire x1="5.715" y1="40.79875" x2="4.92125" y2="40.79875" width="0.127" layer="22"/>
+<wire x1="4.92125" y1="40.79875" x2="4.92125" y2="38.1" width="0.127" layer="22"/>
+<wire x1="4.92125" y1="38.1" x2="5.715" y2="38.1" width="0.127" layer="22"/>
+<text x="4.445" y="40.9575" size="1.27" layer="22" ratio="12" rot="MR270">+5V</text>
 </plain>
 <attributes>
@@
 <elements>
 <element name="C1" library="SMD" package="0805" value="100n" x="13.335" y="31.75" smashed="yes">
-<attribute name="NAME" x="13.589" y="33.401" size="1.016" layer="25" ratio="10"/>
+<attribute name="NAME" x="13.74775" y="34.51225" size="1.016" layer="25" ratio="10"/>
 <attribute name="VALUE" x="11.7475" y="31.3055" size="1.016" layer="27" ratio="10"/>
 </element>
@@
 <attribute name="LAST_DATE_TIME" x="1.27" y="62.38875" size="1.6764" layer="48" font="vector" ratio="12"/>
 </element>
+<element name="U$21" library="Logo" package="OPENHW" value="OPEN_SOURCE_HW" x="14.12875" y="26.51125" smashed="yes" rot="MR0"/>
+<element name="U$22" library="Logo" package="SVEN_TAG" value="" x="8.09625" y="20.47875" smashed="yes" rot="MR0"/>
 </elements>
 <signals>
