File: Rev. 0/Eagle/C64_KernalSw_16k.sch (EAGLE design)
At the start: 8 parts, among them IC1 M27C512-DIP28, IC2 23128SOCKET, IC3 74HCT08D

Commit message: Silk Screen Update
Parts:
- added U$21: OPEN_SOURCE_HW, Logo:OPEN_SOURCE_HW
Other:
- note added: "http://github.com/svenpetersen1965"
Changed lines of the file:
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@@
 <?xml version="1.0" encoding="utf-8"?>
 <!DOCTYPE eagle SYSTEM "eagle.dtd">
-<eagle version="9.2.2">
+<eagle version="9.5.2">
 <drawing>
 <settings>
@@
 <layer number="250" name="Descript" color="7" fill="1" visible="no" active="no"/>
 <layer number="251" name="SMDround" color="7" fill="1" visible="no" active="no"/>
+<layer number="252" name="BR-BS" color="7" fill="1" visible="no" active="yes"/>
+<layer number="253" name="BR-LS" color="7" fill="1" visible="no" active="yes"/>
 <layer number="254" name="OrgLBR" color="7" fill="1" visible="no" active="no"/>
 <layer number="255" name="Accent" color="7" fill="1" visible="yes" active="yes"/>
@@
 <part name="C1" library="SMD" deviceset="C-0805" device="" value="100n"/>
 <part name="U$15" library="!GRAFIK" deviceset="IN" device=""/>
+<part name="U$21" library="Logo" deviceset="OPEN_SOURCE_HW" device=""/>
 </parts>
 <sheets>
@@
 <text x="276.86" y="27.94" size="2.54" layer="95">C64 Kernal Adaptor/Switch</text>
 <text x="276.86" y="22.86" size="2.54" layer="95">for short board (ASSY 250469)</text>
+<text x="279.4" y="7.62" size="2.54" layer="95">http://github.com/svenpetersen1965</text>
 </plain>
 <instances>
@@
 </instance>
 <instance part="U$15" gate="G$1" x="309.88" y="149.86" smashed="yes" rot="R180"/>
+<instance part="U$21" gate="G$1" x="238.76" y="7.62" smashed="yes"/>
 </instances>
 <busses>
